Commit message: Improvements

File: sim/urdf/quadbot.xacro (robot description, xacro)
@@ -1,7 +1,7 @@
 <?xml version="1.0"?>
 <robot name="URDF" xmlns:xacro="http://www.ros.org/wiki/xacro">
-  <xacro:include filename="/home/tomasz/dev/dev_ws/src/quadbot_description/urdf/materials.xacro" />
-  <xacro:include filename="/home/tomasz/dev/dev_ws/src/quadbot_description/urdf/URDF.trans" />
-  <xacro:include filename="/home/tomasz/dev/dev_ws/src/quadbot_description/urdf/URDF.gazebo" />
+  <!-- <xacro:include filename="/home/tomasz/dev/QuadBotNG/sim/urdf/materials.xacro" />
+  <xacro:include filename="/home/tomasz/dev/QuadBotNG/sim/urdf/URDF.trans" /> -->
+  <xacro:include filename="/home/tomasz/dev/QuadBotNG/sim/urdf/URDF.gazebo" />
   <link name="base_link">
     <inertial>
@@ -13,5 +13,5 @@
       <origin xyz="0 0 0" rpy="0 0 0" />
       <geometry>
-        <mesh filename="/home/tomasz/dev/dev_ws/src/quadbot_description/meshes/base_link.stl"
+        <mesh filename="/home/tomasz/dev/QuadBotNG/sim/meshes/base_link.stl"
           scale="0.001 0.001 0.001" />
       </geometry>
@@ -21,5 +21,5 @@
       <origin xyz="0 0 0" rpy="0 0 0" />
       <geometry>
-        <mesh filename="/home/tomasz/dev/dev_ws/src/quadbot_description/meshes/base_link_c.stl"
+        <mesh filename="/home/tomasz/dev/QuadBotNG/sim/meshes/base_link_c.stl"
           scale="0.001 0.001 0.001" />
       </geometry>
@@ -35,5 +35,5 @@
       <origin xyz="-0.039505 -0.0 -0.018083" rpy="0 0 0" />
       <geometry>
-        <mesh filename="/home/tomasz/dev/dev_ws/src/quadbot_description/meshes/drives_1.stl"
+        <mesh filename="/home/tomasz/dev/QuadBotNG/sim/meshes/drives_1.stl"
           scale="0.001 0.001 0.001" />
       </geometry>
@@ -59,5 +59,5 @@
         <origin xyz="-0.039006 ${reflect_y * 0.053} -0.0" rpy="0 0 0" />
         <geometry>
-          <mesh filename="/home/tomasz/dev/dev_ws/src/quadbot_description/meshes/shoulder_${prefix}_1.stl"
+          <mesh filename="/home/tomasz/dev/QuadBotNG/sim/meshes/shoulder_${prefix}_1.stl"
             scale="0.001 0.001 0.001" />
         </geometry>
@@ -68,5 +68,5 @@
         <geometry>
           <mesh
-            filename="/home/tomasz/dev/dev_ws/src/quadbot_description/meshes/shoulder_${prefix}_1_c.stl"
+            filename="/home/tomasz/dev/QuadBotNG/sim/meshes/shoulder_${prefix}_1_c.stl"
             scale="0.001 0.001 0.001" />
         </geometry>
@@ -84,5 +84,5 @@
         <origin xyz="-0.118706 ${reflect_y *0.0875} -0.0" rpy="0 0 0" />
         <geometry>
-          <mesh filename="/home/tomasz/dev/dev_ws/src/quadbot_description/meshes/arm_main_${prefix}_1.stl"
+          <mesh filename="/home/tomasz/dev/QuadBotNG/sim/meshes/arm_main_${prefix}_1.stl"
             scale="0.001 0.001 0.001" />
         </geometry>
@@ -93,5 +93,5 @@
         <geometry>
           <mesh
-            filename="/home/tomasz/dev/dev_ws/src/quadbot_description/meshes/arm_main_${prefix}_1_c.stl"
+            filename="/home/tomasz/dev/QuadBotNG/sim/meshes/arm_main_${prefix}_1_c.stl"
             scale="0.001 0.001 0.001" />
         </geometry>
@@ -108,5 +108,5 @@
         <origin xyz="-0.118706 ${reflect_y *0.0875} -0.0" rpy="0 0 0" />
         <geometry>
-          <mesh filename="/home/tomasz/dev/dev_ws/src/quadbot_description/meshes/arm_crank_${prefix}_1.stl"
+          <mesh filename="/home/tomasz/dev/QuadBotNG/sim/meshes/arm_crank_${prefix}_1.stl"
             scale="0.001 0.001 0.001" />
         </geometry>
@@ -116,5 +116,5 @@
     <origin xyz="-0.118706 0.0875 -0.0" rpy="0 0 0"/>
     <geometry>
-      <mesh filename="/home/tomasz/dev/dev_ws/src/quadbot_description/meshes/arm_crank_${prefix}_1.stl"
+      <mesh filename="/home/tomasz/dev/QuadBotNG/sim/meshes/arm_crank_${prefix}_1.stl"
       scale="0.001 0.001 0.001"/>
     </geometry>
@@ -136,5 +136,5 @@
         <origin xyz="-0.153706 ${reflect_y *0.1026} -0.0" rpy="0 0 0" />
         <geometry>
-          <mesh filename="/home/tomasz/dev/dev_ws/src/quadbot_description/meshes/arm_link_${prefix}_1.stl"
+          <mesh filename="/home/tomasz/dev/QuadBotNG/sim/meshes/arm_link_${prefix}_1.stl"
             scale="0.001 0.001 0.001" />
         </geometry>
@@ -144,5 +144,5 @@
     <origin xyz="-0.153706 0.1026 -0.0" rpy="0 0 0"/>
     <geometry>
-      <mesh filename="/home/tomasz/dev/dev_ws/src/quadbot_description/meshes/arm_link_${prefix}_1.stl"
+      <mesh filename="/home/tomasz/dev/QuadBotNG/sim/meshes/arm_link_${prefix}_1.stl"
       scale="0.001 0.001 0.001"/>
     </geometry>
@@ -165,5 +165,5 @@
         <origin xyz="-0.118702 ${reflect_y *0.1026} 0.119915" rpy="0 0 0" />
         <geometry>
-          <mesh filename="/home/tomasz/dev/dev_ws/src/quadbot_description/meshes/arm_lower_${prefix}_1.stl"
+          <mesh filename="/home/tomasz/dev/QuadBotNG/sim/meshes/arm_lower_${prefix}_1.stl"
             scale="0.001 0.001 0.001" />
         </geometry>
@@ -174,5 +174,5 @@
         <geometry>
           <mesh
-            filename="/home/tomasz/dev/dev_ws/src/quadbot_description/meshes/arm_lower_${prefix}_1_c.stl"
+            filename="/home/tomasz/dev/QuadBotNG/sim/meshes/arm_lower_${prefix}_1_c.stl"
             scale="0.001 0.001 0.001" />
         </geometry>
